Commit message: Changed LiDAR and IMU

File: src/gravel_detect/description/imu.xacro (robot description, xacro)
@@ -2,21 +2,25 @@
 <robot xmlns:xacro="http://www.ros.org/wiki/xacro">
     <link name="imu_link">
-	  <visual>
-		<geometry>
-		  <box size="0.01 0.01 0.005"/>
-		</geometry>
-	  </visual>
-	  <collision>
-		<geometry>
-		  <box size="0.01 0.01 0.005"/>
-		</geometry>
-	  </collision>
-	  <!--<xacro:box_inertia m="0.1" w="0.1" d="0.1" h="0.1"/>-->
-	</link>
-	<joint name="imu_joint" type="fixed">
-	  <parent link="front_right_caster"/>
-	  <child link="imu_link"/>
-	  <origin xyz="0 -0.03 -0.01"/>
-	</joint>
+      <visual>
+        <geometry>
+          <box size="0.01 0.01 0.005"/>
+        </geometry>
+      </visual>
+      <collision>
+        <geometry>
+          <box size="0.01 0.01 0.005"/>
+        </geometry>
+      </collision>
+      <inertial>
+        <mass value="0.01"/>
+        <inertia ixx="0.000001" ixy="0" ixz="0" iyy="0.000001" iyz="0" izz="0.000001"/>
+      </inertial>
+    </link>
+    <!-- IMU mounted directly on base_link for stable reference -->
+    <joint name="imu_joint" type="fixed">
+      <parent link="base_link"/>
+      <child link="imu_link"/>
+      <origin xyz="0.0 0.0 0.1" rpy="0 0 0"/>  <!-- Centered on robot body -->
+    </joint>
   <gazebo reference="imu_link">
     <gravity>true</gravity>

File: src/gravel_detect/description/lidar.xacro (robot description, xacro)
@@ -1,34 +1,33 @@
 <?xml version="1.0"?>
 <robot xmlns:xacro="http://www.ros.org/wiki/xacro">
-    <!-- LiDAR Link -->
-    <link name="lidar_link">
+    <!-- Velodyne LiDAR for iG-LIO compatibility -->
+    <joint name="velodyne_joint" type="fixed">
+        <parent link="base_link"/>
+        <child link="velodyne"/>
+        <origin xyz="0.2 0 0.6" rpy="0 0 0"/>
+    </joint>
+    <link name="velodyne">
         <visual>
             <geometry>
-                <cylinder radius="0.05" length="0.07"/>
+                <cylinder radius="0.052" length="0.072"/>
             </geometry>
-            <material name="black">
-                <color rgba="0.0 0.0 0.0 1.0"/>
+            <material name="velodyne_material">
+                <color rgba="1.0 0.0 0.0 1.0"/>  <!-- Red for visibility -->
             </material>
         </visual>
         <collision>
             <geometry>
-                <cylinder radius="0.05" length="0.07"/>
+                <cylinder radius="0.052" length="0.072"/>
             </geometry>
         </collision>
         <inertial>
-            <mass value="0.5"/>
-            <inertia ixx="0.000732" ixy="0" ixz="0" iyy="0.000732" iyz="0" izz="0.00125"/>
+            <mass value="0.83"/>
+            <origin xyz="0 0 0"/>
+            <inertia ixx="0.001" ixy="0" ixz="0" iyy="0.001" iyz="0" izz="0.001"/>
         </inertial>
     </link>
-    <!-- LiDAR Joint -->
-    <joint name="lidar_joint" type="fixed">
-        <parent link="base_link"/>
-        <child link="lidar_link"/>
-        <origin xyz="0.0 0.0 0.35" rpy="0 0 0"/>
-    </joint>
-    <!-- 3D LiDAR Sensor  -->
-    <gazebo reference="lidar_link">
-        <material>Gazebo/Black</material>
-        <sensor name="lidar_3d" type="ray">
+    <!-- Fixed frame_name to match TF tree -->
+    <gazebo reference="velodyne">
+        <sensor type="ray" name="velodyne_sensor">
             <pose>0 0 0 0 0 0</pose>
             <visualize>true</visualize>
@@ -36,22 +35,20 @@
             <ray>
                 <scan>
-                    <!-- Horizontal scan (360 degrees around) -->
                     <horizontal>
-                        <samples>360</samples>           <!-- 360 beams around -->
+                        <samples>360</samples>
                         <resolution>1</resolution>
-                        <min_angle>-3.14159</min_angle>  <!-- -180° -->
-                        <max_angle>3.14159</max_angle>   <!-- +180° -->
+                        <min_angle>-3.141592654</min_angle>
+                        <max_angle>3.141592654</max_angle>
                     </horizontal>
-                    <!-- Vertical scan (multiple layers) -->
                     <vertical>
-                        <samples>16</samples>            <!-- 16 vertical layers -->
+                        <samples>16</samples>
                         <resolution>1</resolution>
-                        <min_angle>-0.2617</min_angle>   <!-- -15° (down) -->
-                        <max_angle>0.2617</max_angle>    <!-- +15° (up) -->
+                        <min_angle>-0.26</min_angle>
+                        <max_angle>0.26</max_angle>
                     </vertical>
                 </scan>
                 <range>
                     <min>0.1</min>
-                    <max>30.0</max>                      <!-- Good for indoor/outdoor -->
+                    <max>150.0</max>
                     <resolution>0.01</resolution>
                 </range>
@@ -59,16 +56,17 @@
                     <type>gaussian</type>
                     <mean>0.0</mean>
-                    <stddev>0.01</stddev>
+                    <stddev>0.02</stddev>
                 </noise>
             </ray>
-            <!-- 3D Point Cloud Plugin -->
-            <plugin name="lidar_3d_controller" filename="libgazebo_ros_ray_sensor.so">
+            <plugin name="gazebo_ros_ray_sensor" filename="libgazebo_ros_ray_sensor.so">
                 <ros>
-                    <remapping>~/out:=velodyne_points</remapping>  <!-- 3D topic name -->
+                    <namespace></namespace>
+                    <remapping>~/out:=points_raw</remapping>
                 </ros>
-                <output_type>sensor_msgs/PointCloud2</output_type>  <!-- 3D format -->
-                <frame_name>lidar_link</frame_name>
+                <output_type>sensor_msgs/PointCloud2</output_type>
+                <frame_name>velodyne</frame_name>  <!-- Fixed: Use velodyne instead of base_footprint -->
             </plugin>
         </sensor>
+        <material>Gazebo/Red</material>
     </gazebo>
 </robot>

Commit message: Fixed some transforms. Added nav2 package.

File: src/gravel_detect/description/imu.xacro (robot description, xacro)
@@ -75,4 +75,5 @@
                 <remapping>~/out:=data</remapping>
             </ros>
+            <frame_name>imu_link</frame_name>
             <initial_orientation_as_reference>false</initial_orientation_as_reference>
         </plugin>

File: src/gravel_detect/description/robot_core.xacro (robot description, xacro)
@@ -1,5 +1,5 @@
 <?xml version="1.0"?>
 <robot xmlns:xacro="http://www.ros.org/wiki/xacro" name="gravel_detect_robot">
-  <xacro:property name="mesh_path" value="$(find gravel_detect)/meshes/moborobo_short.stl"/>
+  <xacro:property name="mesh_path" value="package://gravel_detect/meshes/moborobo_short.stl"/>
   <link name="base_link">
     <visual>
@@ -124,12 +124,16 @@
   </joint>
   <gazebo>
-    <plugin name="caster_jsp.caster_joint_state_publisher" filename="libgazebo_ros_joint_state_publisher.so">
-      <jointNames>
-        front_caster_1_joint front_caster_1_wheel_joint
-        front_caster_2_joint front_caster_2_wheel_joint
-        back_caster_1_joint back_caster_1_wheel_joint
-        back_caster_2_joint back_caster_2_wheel_joint
-        left_wheel_joint right_wheel_joint
-      </jointNames>
+    <plugin name="gazebo_ros_joint_state_publisher" filename="libgazebo_ros_joint_state_publisher.so">
+      <update_rate>50</update_rate>
+      <joint_name>front_left_caster_joint</joint_name>
+      <joint_name>front_left_caster_wheel_joint</joint_name>
+      <joint_name>front_right_caster_joint</joint_name>
+      <joint_name>front_right_caster_wheel_joint</joint_name>
+      <joint_name>back_left_caster_joint</joint_name>
+      <joint_name>back_left_caster_wheel_joint</joint_name>
+      <joint_name>back_right_caster_joint</joint_name>
+      <joint_name>back_right_caster_wheel_joint</joint_name>
+      <joint_name>left_wheel_joint</joint_name>
+      <joint_name>right_wheel_joint</joint_name>
     </plugin>
   </gazebo>

Commit message: Added stuff to world.

File: src/gravel_detect/description/imu.xacro (robot description, xacro)
@@ -27,5 +27,5 @@
     <sensor name="moborobo_imu" type="imu">
         <always_on>true</always_on>
-        <update_rate>100</update_rate>
+        <update_rate>50</update_rate>
         <imu>
           <angular_velocity>

File: src/gravel_detect/description/lidar.xacro (robot description, xacro)
@@ -22,8 +22,10 @@
         </collision>
         <inertial>
-            <mass value="0.83"/>
-            <origin xyz="0 0 0"/>
-            <inertia ixx="0.001" ixy="0" ixz="0" iyy="0.001" iyz="0" izz="0.001"/>
-        </inertial>
+    <mass value="0.83"/>
+    <origin xyz="0 0 0"/>
+    <inertia ixx="0.00108" ixy="0" ixz="0"
+             iyy="0.00108" iyz="0"
+             izz="0.000562"/>
+    </inertial>
     </link>
     <!-- Use actual Velodyne plugin that includes time and ring fields -->
@@ -36,5 +38,5 @@
                 <scan>
                     <horizontal>
-                        <samples>1800</samples>  <!-- More samples for Velodyne-like behavior -->
+                        <samples>360</samples>  <!-- More samples for Velodyne-like behavior -->
                         <resolution>1</resolution>
                         <min_angle>-3.141592654</min_angle>
@@ -42,5 +44,5 @@
                     </horizontal>
                     <vertical>
-                        <samples>16</samples>   <!-- 16 rings like VLP-16 -->
+                        <samples>8</samples>   <!-- 16 rings like VLP-16 -->
                         <resolution>1</resolution>
                         <min_angle>-0.261799388</min_angle>
