Commit message: fixed transforms and nav params

File: src/gravel_detect/description/controller.xacro (robot description, xacro)
@@ -6,8 +6,9 @@
         <right_joint>right_wheel_joint</right_joint>
         <legacy_mode>false</legacy_mode>
-        <robot_base_frame>base_link</robot_base_frame>
+        <robot_base_frame>base_footprint</robot_base_frame>
         <wheel_separation>0.380</wheel_separation>
         <wheel_diameter>0.2</wheel_diameter>
         <publish_wheel_joint_state>true</publish_wheel_joint_state>
+        <publish_odom_tf>true</publish_odom_tf>
     </plugin>
   </gazebo>

File: src/gravel_detect/description/robot_core.xacro (robot description, xacro)
@@ -1,5 +1,5 @@
 <?xml version="1.0"?>
 <robot xmlns:xacro="http://www.ros.org/wiki/xacro" name="gravel_detect_robot">
-  <xacro:property name="mesh_path" value="package://gravel_detect/meshes/moborobo_short.stl"/>
+  <xacro:property name="mesh_path" value="file://$(find gravel_detect)/meshes/moborobo_short.stl"/>
   <link name="base_link">
     <visual>
@@ -24,5 +24,5 @@
     <parent link="base_footprint"/>
     <child link="base_link"/>
-    <origin xyz="0 0 0" rpy="0 0 0"/>
+    <origin xyz="0 0 0.120" rpy="0 0 0"/>
   </joint>
   <xacro:macro name="caster_wheel" params="caster_name caster_xyz wheel_xyz">
@@ -138,4 +138,5 @@
     </plugin>
   </gazebo>
+  <!-- Gazebo materials -->
   <gazebo reference="back_left_caster"><material>Gazebo/White</material></gazebo>
   <gazebo reference="back_left_caster_wheel"><material>Gazebo/Black</material></gazebo>

Commit message: Improved the world file. Spawn robot at origin. Improved the spacing between the wheels in controller.

File: src/gravel_detect/description/controller.xacro (robot description, xacro)
@@ -7,5 +7,5 @@
         <legacy_mode>false</legacy_mode>
         <robot_base_frame>base_footprint</robot_base_frame>
-        <wheel_separation>0.380</wheel_separation>
+        <wheel_separation>0.350</wheel_separation>
         <wheel_diameter>0.2</wheel_diameter>
         <publish_wheel_joint_state>true</publish_wheel_joint_state>

File: src/gravel_detect/description/lidar.xacro (robot description, xacro)
@@ -22,10 +22,8 @@
         </collision>
         <inertial>
-    <mass value="0.83"/>
-    <origin xyz="0 0 0"/>
-    <inertia ixx="0.00108" ixy="0" ixz="0"
-             iyy="0.00108" iyz="0"
-             izz="0.000562"/>
-    </inertial>
+            <mass value="0.83"/>
+            <origin xyz="0 0 0"/>
+            <inertia ixx="0.001" ixy="0" ixz="0" iyy="0.001" iyz="0" izz="0.001"/>
+        </inertial>
     </link>
     <!-- Use actual Velodyne plugin that includes time and ring fields -->
@@ -38,5 +36,5 @@
                 <scan>
                     <horizontal>
-                        <samples>360</samples>  <!-- More samples for Velodyne-like behavior -->
+                        <samples>1800</samples>  <!-- More samples for Velodyne-like behavior -->
                         <resolution>1</resolution>
                         <min_angle>-3.141592654</min_angle>
@@ -44,5 +42,5 @@
                     </horizontal>
                     <vertical>
-                        <samples>8</samples>   <!-- 16 rings like VLP-16 -->
+                        <samples>16</samples>   <!-- 16 rings like VLP-16 -->
                         <resolution>1</resolution>
                         <min_angle>-0.261799388</min_angle>
